File: 4x6_4/dilemma.kicad_sch (KiCad schematic)
At the start: 342 parts, among them J1 USB_C_Receptacle_USB2.0, J102 NA_serial, J105 NA_Conn_01x04_Female, J113 Cirque, J3 NA_GC9A01, J4 Conn_01x05, J5 NA_Conn_01x02, J5001 USB_C_Receptacle_USB2.0, J5002 NA_Conn_01x02, J5003 NA_serial, J5004 NA_GC9A01, J5005 NA_Conn_01x04_Female, J5007 Cirque, J5008 Conn_01x05, J5009 Conn_01x05, J5010 Conn_01x05, SW1 SW_Push, SW101 NA_SW_Push, SW102 NA_SW_Push, SW103 NA_SW_Push, SW104 NA_SW_Push, SW105 NA_SW_Push, SW106 NA_SW_Push, SW107 NA_SW_Push, SW108 NA_SW_Push, SW109 NA_SW_Push, SW112 NA_SW_Push, SW113 NA_SW_Push, SW114 NA_SW_Push, SW115 NA_SW_Push, SW116 NA_SW_Push, SW117 NA_SW_Push, SW118 NA_SW_Push, SW119 NA_SW_Push, SW3001 NA_SW_Push, SW3002 NA_RotaryEncoder_Switch, SW5001 SW_Push, SW5002 NA_SW_Push, SW5003 NA_SW_Push, SW5004 NA_SW_Push, SW5005 NA_SW_Push, SW5006 NA_SW_Push, SW5007 NA_SW_Push, SW5008 NA_SW_Push, SW5009 NA_SW_Push, SW5010 NA_SW_Push, SW5011 NA_SW_Push, SW5012 NA_SW_Push, SW5013 NA_SW_Push, SW5014 NA_SW_Push, SW5015 NA_SW_Push, SW5016 NA_SW_Push, SW5017 NA_SW_Push, SW5018 NA_SW_Push, SW5019 NA_SW_Push, SW5020 NA_RotaryEncoder_Switch, SW5021 SW_SPST, SW5022 SW_SPST, SW5023 NA_SW_Push, SW5024 NA_SW_Push, SW5025 NA_SW_Push, SW5026 NA_SW_Push, SW5027 NA_SW_Push, SW5028 NA_SW_Push, SW5029 NA_SW_Push, SW5030 NA_SW_Push, SW5031 NA_SW_Push, SW5032 NA_SW_Push, SW5033 NA_SW_Push, SW5034 NA_SW_Push, SW5035 NA_SW_Push, SW5036 NA_SW_Push, SW5037 NA_SW_Push, SW5038 NA_SW_Push, SW5039 NA_SW_Push, SW5040 NA_SW_Push, SW5041 NA_SW_Push, SW5042 NA_SW_Push, U1 RP2040, U2 W25Q128JVS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

Commit message: added vik support to schematic for dilemma v3, along with initial part placement and routing
Parts:
- removed J113, J5007: Cirque, local-libraries:FPC-SMD_FPC05012-09200-.5mm, symbol Connector:Conn_01x14_Female
- added J5006, J5007: ~, vik:vik-module-connector-horizontal, symbol vik:vik-module-connector
- added JP5001, JP5002: SolderJumper_3_Bridged12, Jumper:SolderJumper-3_P1.3mm_Bridged12_RoundedPad1.0x1.5mm, symbol Jumper:SolderJumper_3_Bridged12
- added SW5043, SW5044: SW_SPDT, local-libraries:MSK-12C02, symbol Switch:SW_SPDT
Connections:
- net +3V3: now also R103.1, J5006.12 (3V3); no longer R103.2
- net +3V3_L: now also J5007.12 (3V3)
- net +5V: now also SW5044.1 (A)
- net +5V_L: now also SW5043.1 (A)
- net GND: now also J5006.11 (GND)
- net GND_L: now also J5007.11 (GND)
- net MISO: now also J5006.2 (MISO)
- net MISO_L: now also J5007.2 (MISO)
- net MOSI: now also J5006.5 (MOSI)
- net MOSI_L: now also J5007.5 (MOSI)
- net NCS: now also J5006.3 (SPI_CS)
- net NCS_L: now also J5007.3 (SPI_CS)
- net RGB: now also JP5001.2 (C); no longer D5109.3 (DOUT)
- net RGB_L: now also JP5002.2 (C); no longer D5113.3 (DOUT)
- net SCL: now also J5006.9 (SCL)
- net SCLK: now also J5006.1 (SCLK)
- net SCLK_L: now also J5007.1 (SCLK)
- net SCL_L: now also J5007.9 (SCL)
- net SDA: now also R103.2, J5006.10 (SDA); no longer R103.1
- net SDA_L: now also J5007.10 (SDA)
- net VIK_RGB: now reaches D5127.1 (DOUT)
- net VIK_RGB: now also J5006.8 (RGB_LED_IN), JP5001.3 (B)
- net VIK_RGB_L: now reaches D5137.1 (DOUT)
- net VIK_RGB_L: now also J5007.8 (RGB_LED_IN), JP5002.3 (B)
- net QP_CS renamed VIK_GP1
- net VIK_GP1: now also J5006.6 (GPIO_AD1)
- net QP_CS_L renamed VIK_GP1_L
- net VIK_GP1_L: now also J5007.6 (GPIO_AD1)
- net QP_DC renamed VIK_GP2
- net VIK_GP2: now also J5006.4 (GPIO_AD2)
- net QP_DC_L renamed VIK_GP2_L
- net VIK_GP2_L: now also J5007.4 (GPIO_AD2)
- new net: J5007.7 (5V), SW5043.2 (B)
- new net: J5006.7 (5V), SW5044.2 (B)
- new net: D5113.3 (DOUT), JP5002.1 (A)
- new net: D5109.3 (DOUT), JP5001.1 (A)
- no-connect marks 27 -> 14
Other:
- moved on the sheet: C5017, C5018, D5031, D5032, D5033, D5034, D5035, D5036, D5037, D5038, D5039, D5040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
